File: SSD1303_Breakout.kicad_pcb (KiCad board)
At the start: 2 copper layers, 62.5 x 49.5 mm, 64 parts, among them J1 PinHeader, Q1 2N7002, Q2 2N7002, U1 TPS61040DBV, U2 XC6206P332MR

Commit message: final™ touches
Parts:
- removed JP1: PAR/~{SER}, Jumper:SolderJumper-2_P1.3mm_Open_TrianglePad1.0x1.5mm
- removed kibuzzard-64927BC4: G***, kibuzzard-64927BC4
- removed kibuzzard-64927C10: G***, kibuzzard-64927C10
- removed kibuzzard-64927C21: G***, kibuzzard-64927C21
- removed kibuzzard-64927C38: G***, kibuzzard-64927C38
- moved REF** 3.44 mm to (97.0, 99.2)
Connections:
- net OLED_BS2 renamed /OLED_BS2
Routing:
- net +3V3: track 110.2 -> 109.3 mm
Other:
- outline, holes or cut-outs redrawn
- board text added: "I2C"
- board text added: "SPI"
