File: SSD1303_Breakout.kicad_sch (KiCad schematic)
At the start: 36 parts, among them J1 PinHeader, Q1 2N7002, Q2 2N7002, U1 TPS61040DBV, U2 XC6206P332MR

Commit message: final™ touches
Parts:
- removed JP1: PAR/~{SER}, Jumper:SolderJumper-2_P1.3mm_Open_TrianglePad1.0x1.5mm, symbol Jumper:SolderJumper_2_Open
Other:
- moved on the sheet: C1, R13
